Commit message: Regenerate scara urdf

File: urdf/kits/HEBI_Scara.urdf (robot description, URDF)
Before this commit: robot HEBI_Scara, 7 links, 6 joints
Links:
- added link HEBI_SIM/Arm/J1_shoulder/X8_9, mass 0.001; visual sphere radius=0.001
- added link HEBI_SIM/Arm/J2_elbow/X8_9, mass 0.001; visual sphere radius=0.001
- added link HEBI_SIM/Arm/J3_wrist/X8_9, mass 0.001; visual sphere radius=0.001
- link end_effector/INPUT_INTERFACE: mass 0.02 -> 0.2; geometry visual box rpy=0 0 0 size=0.001 0.001 0.001
Joints:
- removed joint Arm/J1_shoulder/X8_9
- removed joint Arm/J2_elbow/X8_9
- removed joint Arm/J3_wrist/X8_9
- added joint Arm/J1_shoulder: type continuous, parent Arm/J1_shoulder/INPUT_INTERFACE, child shoulder_elbow/INPUT_INTERFACE, origin xyz=0 0 0.045 rpy=0 0 0, axis 0 0 1, limit effort=20 velocity=30
- added joint Arm/J2_elbow: type continuous, parent Arm/J2_elbow/INPUT_INTERFACE, child elbow_wrist/INPUT_INTERFACE, origin xyz=0 0 0.045 rpy=0 0 0, axis 0 0 1, limit effort=20 velocity=30
- added joint Arm/J3_wrist: type continuous, parent Arm/J3_wrist/INPUT_INTERFACE, child end_effector/INPUT_INTERFACE, origin xyz=0 0 0.045 rpy=0 0 0, axis 0 0 1, limit effort=20 velocity=30
- added joint HEBI_SIM_JOINT/Arm/J1_shoulder: type fixed, parent Arm/J1_shoulder/INPUT_INTERFACE, child HEBI_SIM/Arm/J1_shoulder/X8_9, origin xyz=0 0 0 rpy=0 0 0
- added joint HEBI_SIM_JOINT/Arm/J2_elbow: type fixed, parent Arm/J2_elbow/INPUT_INTERFACE, child HEBI_SIM/Arm/J2_elbow/X8_9, origin xyz=0 0 0 rpy=0 0 0
- added joint HEBI_SIM_JOINT/Arm/J3_wrist: type fixed, parent Arm/J3_wrist/INPUT_INTERFACE, child HEBI_SIM/Arm/J3_wrist/X8_9, origin xyz=0 0 0 rpy=0 0 0
