Commit message: Add visual and collision to rail of Scara_ext

File: urdf/kits/HEBI_Scara_ext.urdf (robot description, URDF)
Before this commit: robot HEBI_Scara, 11 links, 10 joints
Links:
- link rail: mass None -> 1; geometry collision cylinder length=2 radius=.016; visual cylinder length=2 radius=.016
